File: RotaryRemotePCB.kicad_pcb (KiCad board)
At the start: 2 copper layers, 59 x 55 mm, 12 parts, among them J3 i2c, J4 Neopixel Connector, J5 EncoderRotary, J6 EncoderSwitch, SW2 SW_SPST, U1 TP4056, U2 WeMos_D1_mini, U3 magnetic-charger, U4 TTL

Commit message: Rearrange the sockets
Parts:
- moved BT1 32.8 mm to (132.2, 112.0), turned to 180 degrees
- moved J4 12.0 mm to (107.6, 78.5), turned to 0 degrees
- moved SW2 4.00 mm to (122.0, 115.0)
Routing:
- net /VBAT: track 5.39 -> 36.8 mm
- net /VBAT-: track 5.73 -> 27.3 mm
- net Net-(J4-Pad2): track 23.9 -> 12.7 mm
- net +5V: track 59.6 -> 56.1 mm
- net +3V3: track 108.2 -> 106.5 mm
- net /5V: track 31.0 -> 29.4 mm
Other:
- outline, holes or cut-outs redrawn
